Commit message: map OK

File: src/visual_robot/urdf/ahpu_robot.urdf (robot description, URDF)
Before this commit: robot four_wheel_robot, 5 links, 4 joints
Links:
- added link laser; visual cylinder length=0.1 radius=0.05
Joints:
- added joint laser_joint: type fixed, parent base_link, child laser, origin xyz=0.2 0 0.15 rpy=0 0 0

Commit message: visualtest

File: src/visual_robot/urdf/ahpu_robot.urdf (robot description, URDF)
Before this commit: robot four_wheel_robot, 6 links, 5 joints
Links:
- removed link laser
- added link laser_link; visual cylinder length=0.1 radius=0.05
Joints:
- joint laser_joint: child laser -> laser_link
